File: audio_out.kicad_sch (KiCad schematic)
At the start: 44 parts, among them J3 LINEOUT, J4 SPKRL, J5 SPKRR, J6 HPOUT, Q1 BSS138, Q2 BSS138, U5 PAM8019

Commit message: Initial schematic of Rev3.
Parts:
- removed C28, C30, C32: 1uF, Capacitor_SMD:C_0805_2012Metric_Pad1.18x1.45mm_HandSolder, symbol Device:C_Small
- removed C29, C31, C38: 0.1uF, Capacitor_SMD:C_0805_2012Metric_Pad1.18x1.45mm_HandSolder, symbol Device:C_Small
- removed C33, C35: 10uF, Capacitor_SMD:C_0805_2012Metric_Pad1.18x1.45mm_HandSolder, symbol Device:C_Small
- removed C34: 2.2uF, Capacitor_SMD:C_0805_2012Metric_Pad1.18x1.45mm_HandSolder, symbol Device:C_Small
- removed C36, C37: 220uF, Capacitor_SMD:CP_Elec_6.3x5.4, symbol Device:C_Polarized_Small
- removed C39, C40, C41, C42: 200pF, Capacitor_SMD:C_0805_2012Metric_Pad1.18x1.45mm_HandSolder, symbol Device:C_Small
- removed FB2: FSPKRR+, Resistor_SMD:R_0805_2012Metric_Pad1.20x1.40mm_HandSolder, symbol Device:FerriteBead_Small
- removed FB3: FSPKRR-, Resistor_SMD:R_0805_2012Metric_Pad1.20x1.40mm_HandSolder, symbol Device:FerriteBead_Small
- removed FB4: FSPKRL+, Resistor_SMD:R_0805_2012Metric_Pad1.20x1.40mm_HandSolder, symbol Device:FerriteBead_Small
- removed FB5: FSPKRL-, Resistor_SMD:R_0805_2012Metric_Pad1.20x1.40mm_HandSolder, symbol Device:FerriteBead_Small
- removed J3: LINEOUT, pico_synth_sandbox:Jack_3.5mm_PJ327A_Horizontal, symbol Connector_Audio:AudioJack4_SwitchT1
- removed JP9: MUTE_ENABLE, Jumper:SolderJumper-3_P1.3mm_Bridged12_RoundedPad1.0x1.5mm, symbol Jumper:SolderJumper_3_Bridged12
- removed Q1, Q2: BSS138, Package_TO_SOT_SMD:SOT-23, symbol Transistor_FET:BSS138
- removed R10, R11, R12: NC, Resistor_SMD:R_0805_2012Metric_Pad1.20x1.40mm_HandSolder, symbol Device:R_Small
- removed R13, R14, R8, R9: 100k, Resistor_SMD:R_0805_2012Metric_Pad1.20x1.40mm_HandSolder, symbol Device:R_Small
- removed R5: 10k, Resistor_SMD:R_0805_2012Metric_Pad1.20x1.40mm_HandSolder, symbol Device:R_Small
- removed R6: 1k, Resistor_SMD:R_0805_2012Metric_Pad1.20x1.40mm_HandSolder, symbol Device:R_Small
- removed R7: 2.4k, Resistor_SMD:R_0805_2012Metric_Pad1.20x1.40mm_HandSolder, symbol Device:R_Small
- removed RV3: 10k, pico_synth_sandbox:RK10J12R0A0B, symbol pico_synth_sandbox:RK10J12R0A0B
- removed U5: PAM8019, Package_DFN_QFN:QFN-20-1EP_4x4mm_P0.5mm_EP2.5x2.5mm, symbol pico_synth_sandbox:PAM8019
Connections:
- net AMPL+: no longer names the net of J4.1 (Pin_1), TP6.1
- net AMPL-: no longer names the net of J4.2 (Pin_2), TP7.1
- net AMPR+: no longer names the net of J5.1 (Pin_1), TP8.1
- net AMPR-: no longer names the net of J5.2 (Pin_2), TP9.1
- net GND renamed HP_G
- net HPL_OUT renamed HP_L
- net HPR_OUT renamed HP_R
- no-connect marks 4 -> 1
Other:
- note removed: "Line Output"
- note removed: "vUVP = (1.2-(6uF*R3))*(R1+R2)/R2 Hysteresis = 5uF*R3*(R1+R2)/R2"
