File: battery.kicad_sch (KiCad schematic)
At the start: 17 parts, among them Q3 BSS84, Q4 BSS84, Q5 BSS138, Q6 BSS138, U6 MCP73831-5-OT, U7 AP9101CK6

Commit message: Initial schematic of Rev3.
Parts:
- removed C43: 10uF, Capacitor_SMD:C_0805_2012Metric_Pad1.18x1.45mm_HandSolder, symbol Device:C_Small
- removed C45: 0.1uF, Capacitor_SMD:C_0805_2012Metric_Pad1.18x1.45mm_HandSolder, symbol Device:C_Small
- removed Q3, Q4: BSS84, Package_TO_SOT_SMD:SOT-23_Handsoldering, symbol Transistor_FET:BSS84
- removed Q5, Q6: BSS138, Package_TO_SOT_SMD:SOT-23_Handsoldering, symbol Transistor_FET:BSS138
- removed R15: 1k, Resistor_SMD:R_0805_2012Metric_Pad1.20x1.40mm_HandSolder, symbol Device:R_Small
- removed R18: 330, Resistor_SMD:R_0805_2012Metric_Pad1.20x1.40mm_HandSolder, symbol Device:R_Small
- removed R19: 2.7k, Resistor_SMD:R_0805_2012Metric_Pad1.20x1.40mm_HandSolder, symbol Device:R_Small
- removed U7: AP9101CK6, Package_TO_SOT_SMD:SOT-23-6, symbol Battery_Management:AP9101CK6
- added C5, C6, C7, C8, C9: 10uF, Capacitor_SMD:C_0805_2012Metric_Pad1.18x1.45mm_HandSolder, symbol Device:C_Small
- added D6: MBR0540, Diode_SMD:D_SOD-123, symbol Diode:MBR0540
- added D7: PWR, LED_SMD:LED_0805_2012Metric_Pad1.15x1.40mm_HandSolder, symbol Device:LED
- added Q1: DMG3415, Package_TO_SOT_SMD:SOT-23_Handsoldering, symbol Transistor_FET:BSS84
- added R1, R2, R4, R5: 10k, Resistor_SMD:R_0805_2012Metric_Pad1.20x1.40mm_HandSolder, symbol Device:R_Small
- added SW4: SW_SPDT, symbol Switch:SW_SPDT
- added U1, U3: AP2112K-3.3, Package_TO_SOT_SMD:SOT-23-5, symbol Regulator_Linear:AP2112K-3.3
- R16: value 4.7k -> 5.1k
- R17: value 1k -> 10k
Connections:
- net -BATT is gone; now on net GND: BT1.2 (-)
- net GND: now also C5.2, C6.2, C7.2, C8.2, C9.2, R1.2, R2.2, R4.2, SW4.3 (C), U1.2 (GND), U3.2 (GND)
- net VBUS: now also D2.2 (A), C5.1, D6.2 (A), Q1.1 (G), R1.1; no longer D2.1 (K)
- net VSYS: now also C6.1, C9.1, D6.1 (K), Q1.2 (S), R5.1, U1.1 (VIN), U3.1 (VIN)
- net at R17.1: now also D2.1 (K); no longer D2.2 (A)
- net VDD: now reaches D1.2 (A)
- net VDD: now also C7.1, U3.5 (VOUT)
- net +3.3V: no longer names the net of D1.1 (K)
- net +3.3V: now also R4.1
- net +BATT renamed VBAT
- net VBAT: now also Q1.3 (D)
- new net: D7.1 (K), R2.1
- new net PWR_EN: R5.2, SW4.2 (B), U1.3 (EN), U3.3 (EN)
- new net VDDA: C8.1, D7.2 (A), U1.5 (VOUT)
Other:
- note added: "Analog Power Regulation"
- note added: "Battery Charging"
- note added: "Digital Power Regulation"
- note added: "VSYS"
- note removed: "VBAT and +BATT are the same"
- note removed: "VBUS/VBAT Power Switching and Power Enable Switch"
- moved on the sheet: BT1, C44, R16, R17, U6
