File: i2s_adc.kicad_sch (KiCad schematic)
At the start: 28 parts, among them J2 LINEIN, U4 PCM1860DBTR

Commit message: Initial schematic of Rev3.
Parts:
- removed C15, C17, C26, C27: 0.1uF, Capacitor_SMD:C_0805_2012Metric_Pad1.18x1.45mm_HandSolder, symbol Device:C_Small
- removed C16, C18, C20, C21, C22, C23: 10uF, Capacitor_SMD:C_0805_2012Metric_Pad1.18x1.45mm_HandSolder, symbol Device:C_Small
- removed C19: 1uF, Capacitor_SMD:C_0805_2012Metric_Pad1.18x1.45mm_HandSolder, symbol Device:C_Small
- removed C24, C25: 2.2uF, Capacitor_SMD:C_0805_2012Metric_Pad1.18x1.45mm_HandSolder, symbol Device:C_Small
- removed J2: LINEIN, pico_synth_sandbox:Jack_3.5mm_PJ327A_Horizontal, symbol Connector_Audio:AudioJack4_SwitchT1
- removed JP6: FILT, Jumper:SolderJumper-2_P1.3mm_Open_RoundedPad1.0x1.5mm, symbol Jumper:SolderJumper_2_Open
- removed JP7: MIC_GAIN_0, Jumper:SolderJumper-2_P1.3mm_Bridged_RoundedPad1.0x1.5mm, symbol Jumper:SolderJumper_2_Bridged
- removed JP8: MIC_GAIN_32, Jumper:SolderJumper-2_P1.3mm_Open_RoundedPad1.0x1.5mm, symbol Jumper:SolderJumper_2_Open
- removed MK1: MIC_L, pico_synth_sandbox:Knowles_SPU0410HR5H-PB_3.76x2.95mm, symbol pico_synth_sandbox:SPU0410HR5H
- removed MK2: MIC_R, pico_synth_sandbox:Knowles_SPU0410HR5H-PB_3.76x2.95mm, symbol pico_synth_sandbox:SPU0410HR5H
- removed R3: 1k, Resistor_SMD:R_0805_2012Metric_Pad1.20x1.40mm_HandSolder, symbol Device:R_Small
- removed R4: 10k, Resistor_SMD:R_0805_2012Metric_Pad1.20x1.40mm_HandSolder, symbol Device:R_Small
- removed RN4: 10k, Resistor_SMD:R_Array_Convex_4x1206, symbol Device:R_Pack04
- removed RN5: 22, Resistor_SMD:R_Array_Convex_4x1206, symbol Device:R_Pack04
- removed RV2: 10k, pico_synth_sandbox:RK10J12R0A0B, symbol pico_synth_sandbox:RK10J12R0A0B
- removed TP26: MIC_L, TestPoint:TestPoint_Pad_D2.0mm, symbol Connector:TestPoint
- removed TP27: MIC_R, TestPoint:TestPoint_Pad_D2.0mm, symbol Connector:TestPoint
- removed TP5: SCK, TestPoint:TestPoint_Pad_D2.0mm, symbol Connector:TestPoint
- removed U4: PCM1860DBTR, Package_SO:TSSOP-30_4.4x7.8mm_P0.5mm, symbol pico_synth_sandbox:PCM1860DBTR
Connections:
- no-connect marks 3 -> 0
Other:
- note removed: "ADC"
- note removed: "Line Input"
- note removed: "Not sure about the implementation of INT here. Maybe GND it?"
- note removed: "Power Filtering"
- note removed: "Stereo Microphones"
