File: keyboard.kicad_sch (KiCad schematic)
At the start: 35 parts, among them U8 TTP229-BSF

Commit message: Initial schematic of Rev3.
Parts:
- removed C46, C47, C48, C49, C50, C51: 0-50pF, Capacitor_SMD:C_0805_2012Metric_Pad1.18x1.45mm_HandSolder, symbol Device:C_Variable
- removed C52: 0.1uF, Capacitor_SMD:C_0805_2012Metric_Pad1.18x1.45mm_HandSolder, symbol Device:C_Small
- removed C53: 10uF, Capacitor_SMD:C_0805_2012Metric_Pad1.18x1.45mm_HandSolder, symbol Device:C_Small
- removed JP10: OPDEN, Jumper:SolderJumper-2_P1.3mm_Open_RoundedPad1.0x1.5mm, symbol Jumper:SolderJumper_2_Open
- removed JP11: SAHL, Jumper:SolderJumper-2_P1.3mm_Bridged_RoundedPad1.0x1.5mm, symbol Jumper:SolderJumper_2_Bridged
- removed JP12: KYSEL, Jumper:SolderJumper-2_P1.3mm_Bridged_RoundedPad1.0x1.5mm, symbol Jumper:SolderJumper_2_Bridged
- removed JP13: SKMS1, Jumper:SolderJumper-2_P1.3mm_Bridged_RoundedPad1.0x1.5mm, symbol Jumper:SolderJumper_2_Bridged
- removed JP14: SKMS0, Jumper:SolderJumper-2_P1.3mm_Bridged_RoundedPad1.0x1.5mm, symbol Jumper:SolderJumper_2_Bridged
- removed JP15: WPSCT, Jumper:SolderJumper-2_P1.3mm_Open_RoundedPad1.0x1.5mm, symbol Jumper:SolderJumper_2_Open
- removed JP16: SLWPTM, Jumper:SolderJumper-2_P1.3mm_Open_RoundedPad1.0x1.5mm, symbol Jumper:SolderJumper_2_Open
- removed JP17: SKSRT, Jumper:SolderJumper-2_P1.3mm_Open_RoundedPad1.0x1.5mm, symbol Jumper:SolderJumper_2_Open
- removed RN6, RN7: 1M, Resistor_SMD:R_Array_Convex_4x1206, symbol Device:R_Pack04
- removed U8: TTP229-BSF, Package_SO:SSOP-28_3.9x9.9mm_P0.635mm, symbol pico_synth_sandbox:TTP229-BSF
- added R10, R11, R12, R13, R14, R15, R18, R19, R26, R27, R28, R29, R6, R7, R8, R9: 1M, symbol Device:R_Small
Connections:
- net GND: now also R10.1, R11.1, R12.1, R13.1, R14.1, R15.1, R18.1, R19.1, R26.1, R27.1, R28.1, R29.1, R6.1, R7.1, R8.1, R9.1
- net TPAD10: now also R18.2
- net TPAD11: now also R19.2
- net TPAD12: now also R26.2
- net TPAD13: now also R27.2
- net TPAD14: now also R28.2
- net TPAD15: now also R29.2
- net TPAD5: now also R11.2
- net TPAD8: now also R14.2
- net TPAD9: now also R15.2
- net KYSEL renamed TPAD2
- net TPAD2: now also R8.2
- net OPDEN renamed TPAD0
- net TPAD0: now also R6.2
- net SAHL renamed TPAD1
- net TPAD1: now also R7.2
- net SKMS0 renamed TPAD4
- net TPAD4: now also R10.2
- net SKMS1 renamed TPAD3
- net TPAD3: now also R9.2
- net SKSRT renamed TPAD7
- net TPAD7: now also R13.2
- net SLWPTM renamed TPAD6
- net TPAD6: now also R12.2
