File: power.kicad_sch (KiCad schematic)
At the start: 0 parts

Commit message: Initial schematic of Rev3.
Other:
- title: pico_synth_sandbox - MIDI Input & Output -> pico_synth_sandbox - LiPo Battery Power & Charging
Changed lines of the file:
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@@
 	(paper "A")
 	(title_block
-		(title "pico_synth_sandbox - MIDI Input & Output")
+		(title "pico_synth_sandbox - LiPo Battery Power & Charging")
 		(date "2024-09-08")
 		(rev "3")
