File: codec.kicad_sch (KiCad schematic)
At the start: 49 parts, among them J2 LINEIN, J6 HPOUT, U2 WM8960CGEFL/V, X1 ECS-2520MV-240-BN-TR

Commit message: Rename "pico_synth_sandbox" to "PicoSynth_Sandbox"
Parts:
- J2, J6: footprint pico_synth_sandbox:Jack_3.5mm_PJ327A_Horizontal -> PicoSynth_Sandbox:Jack_3.5mm_PJ327A_Horizontal
- U2: symbol pico_synth_sandbox:WM8960CGEFL/V -> PicoSynth_Sandbox:WM8960CGEFL/V
Other:
- title: pico_synth_sandbox - Audio Output -> PicoSynth_Sandbox - Audio Output
