File: PicoSynth_Sandbox.kicad_sch (KiCad schematic)
At the start: 58 parts, among them J1 Micro_SD_Card_Det2, J3 MIDIIN, J4 MIDIOUT, Q2 DMG3415, SW3 PWR, U1 MAX17048, U12 Pico, U3 AP2112K-3.3, U5 H11L1, U6 MCP73831-5-OT

Commit message: Board outline.
Parts:
- H1, H2, H3, H4: footprint MountingHole:MountingHole_2.5mm_Pad -> MountingHole:MountingHole_3.2mm_M3_Pad_TopOnly
Changed lines of the file:
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@@
 			)
 		)
-		(property "Footprint" "MountingHole:MountingHole_2.5mm_Pad"
+		(property "Footprint" "MountingHole:MountingHole_3.2mm_M3_Pad_TopOnly"
 			(at 247.65 158.75 0)
 			(effects
@@
 			)
 		)
-		(property "Footprint" "MountingHole:MountingHole_2.5mm_Pad"
+		(property "Footprint" "MountingHole:MountingHole_3.2mm_M3_Pad_TopOnly"
 			(at 247.65 144.78 0)
 			(effects
@@
 			)
 		)
-		(property "Footprint" "MountingHole:MountingHole_2.5mm_Pad"
+		(property "Footprint" "MountingHole:MountingHole_3.2mm_M3_Pad_TopOnly"
 			(at 256.54 158.75 0)
 			(effects
@@
 			)
 		)
-		(property "Footprint" "MountingHole:MountingHole_2.5mm_Pad"
+		(property "Footprint" "MountingHole:MountingHole_3.2mm_M3_Pad_TopOnly"
 			(at 256.54 144.78 0)
 			(effects
