File: touch.kicad_sch (KiCad schematic)
At the start: 80 parts, among them SW1 RotaryEncoder_Switch, SW2 RotaryEncoder_Switch, U10 MPR121QR2, U11 MPR121QR2, U9 MPR121QR2

Commit message: Rename "pico_synth_sandbox" to "PicoSynth_Sandbox"
Parts:
- TP10: footprint pico_synth_sandbox:CapKeysWhite -> PicoSynth_Sandbox:CapKeysWhite
- TP11, TP16, TP23: footprint pico_synth_sandbox:CapKeysWhiteLeft -> PicoSynth_Sandbox:CapKeysWhiteLeft
- TP12, TP14, TP17, TP19, TP21, TP24, TP30, TP32, TP7, TP9: footprint pico_synth_sandbox:CapKeysBlack -> PicoSynth_Sandbox:CapKeysBlack
- TP13, TP18, TP20: footprint pico_synth_sandbox:CapKeysWhiteMiddle -> PicoSynth_Sandbox:CapKeysWhiteMiddle
- TP15, TP22, TP25, TP26, TP31, TP33, TP8: footprint pico_synth_sandbox:CapKeysWhiteRight -> PicoSynth_Sandbox:CapKeysWhiteRight
Other:
- title: pico_synth_sandbox - Touch Keyboard -> PicoSynth_Sandbox - Touch Keyboard

Commit message: Board outline.
Parts:
- removed R67, R68, R69, R70, R71, R72, R73, R74: 1M, symbol Device:R
- removed SW1, SW2: RotaryEncoder_Switch, Rotary_Encoder:RotaryEncoder_Alps_EC11E-Switch_Vertical_H20mm, symbol Device:RotaryEncoder_Switch
- added R16, R17, R5, R58: 1M, symbol Device:R
- added TP34: TCH3, symbol Connector:TestPoint
- added TP35: TCH4, symbol Connector:TestPoint
- TP30: value C#4/Db4 -> BTN1; footprint PicoSynth_Sandbox:CapKeysBlack -> (none)
- TP31: value D4 -> TCH0; footprint PicoSynth_Sandbox:CapKeysWhiteRight -> (none)
- TP32: value C#4/Db4 -> TCH1; footprint PicoSynth_Sandbox:CapKeysBlack -> (none)
- TP33: value D4 -> TCH2; footprint PicoSynth_Sandbox:CapKeysWhiteRight -> (none)
- TP7: value C#4/Db4 -> VAL2; footprint PicoSynth_Sandbox:CapKeysBlack -> (none)
- TP8: value D4 -> VAL1; footprint PicoSynth_Sandbox:CapKeysWhiteRight -> (none)
- TP9: value C#4/Db4 -> VAL0; footprint PicoSynth_Sandbox:CapKeysBlack -> (none)
Connections:
- net BTN0: now also TP26.1, U10.12 (LED0/ELE4), R58.2; no longer U11.18 (LED6/ELE10)
- net GND: now also R16.2, R17.2, R5.2, R58.1
- net MOD0: now also U11.8 (ELE0); no longer U11.11 (ELE3)
- net MOD1: now also U11.9 (ELE1); no longer U11.12 (LED0/ELE4)
- net MOD2: now also U11.10 (ELE2); no longer U11.13 (LED1/ELE5)
- net PTCH0: now also U10.17 (LED5/ELE9); no longer U11.8 (ELE0)
- net PTCH1: now also U10.18 (LED6/ELE10); no longer U11.9 (ELE1)
- net PTCH2: now also U10.19 (LED7/ELE11); no longer U11.10 (ELE2)
- net WHL0: now also U11.11 (ELE3); no longer U11.14 (LED2/ELE6)
- net WHL1: now also U11.12 (LED0/ELE4); no longer U11.15 (LED3/ELE7)
- net WHL2: now also U11.13 (LED1/ELE5); no longer U11.16 (LED4/ELE8)
- net WHL3: now also U11.14 (LED2/ELE6); no longer U11.17 (LED5/ELE9)
- net BTN1: no longer names the net of U11.19 (LED7/ELE11)
- net BTN1: now also TP35.1
- net KEY16 renamed VAL2
- net VAL2: now also U10.16 (LED4/ELE8), R5.1; no longer U10.12 (LED0/ELE4)
- net KEY17: no longer names the net of U10.13 (LED1/ELE5)
- net KEY17: now also TP30.1; no longer TP8.1
- net KEY18 renamed VAL0
- net VAL0: now also R17.1
- net KEY19 renamed VAL1
- net VAL1: now also TP8.1, R16.1; no longer TP26.1
- removed net KEY20: TP30.1, U10.16 (LED4/ELE8)
- net KEY21: no longer names the net of TP31.1
- net KEY21: now also U11.15 (LED3/ELE7); no longer U10.17 (LED5/ELE9)
- net KEY22: no longer names the net of TP32.1
- net KEY22: now also U11.16 (LED4/ELE8); no longer U10.18 (LED6/ELE10)
- net KEY23: no longer names the net of TP33.1
- net KEY23: now also U11.17 (LED5/ELE9); no longer U10.19 (LED7/ELE11)
- new net: TP34.1, U11.18 (LED6/ELE10)
Other:
- note removed: "Encoders"
